File: board/stm-universal-can-board/stm-universal-can-board.sch (KiCad schematic (older format))
At the start: 5 parts

Commit message: Continued STM Board development
Parts:
- removed U?: MCP2551-I-SN, Package_SO:SOIC-8_3.9x4.9mm_P1.27mm, symbol Interface_CAN_LIN:MCP2551-I-SN
- added C?: 100n, symbol Device:C
- added C?: 47u, symbol Device:CP
- added C?: C, symbol Device:C
- added C? (x2): 47pF, symbol Device:C
- added C?: 10nF, symbol Device:C
- added D?: B2100-13-F, symbol Device:D_Schottky
- added J?: USB_OTG, symbol Connector:USB_OTG
- added J?: Conn_01x02, symbol Connector_Generic:Conn_01x02
- added JP?: Jumper, symbol Jumper:Jumper_3_Bridged12
- added R? (x2): 27R, symbol Device:R
- added U?: SN65HVD230, Package_SO:SOIC-8_3.9x4.9mm_P1.27mm, symbol Interface_CAN_LIN:SN65HVD230
Connections:
- net labels added: +12V, +5V, D+, D-, GND, VBUS, VCC
- wire segments 0 -> 46
- no-connect marks 0 -> 1
Other:
- note added: "Power Management"
- moved on the sheet: U?

Commit message: Added comments and continued design (USB-UART converter)
Parts:
- removed C?: 47u, symbol Device:CP
- removed C? (x2): 47pF, symbol Device:C
- removed R? (x2): 27R, symbol Device:R
- added C? (x2): 4u7, symbol Device:C
- added C? (x2): 100n, symbol Device:C
- added D?: B2100-13-F, symbol Device:D_Schottky
- added D? (x2): LED, symbol Device:LED
- added R? (x2): R??, symbol Device:R
- C?: value 10nF -> 100n
Connections:
- net labels added: RESET, USB_RX, USB_TX
- net labels removed: +5V
- wire segments 46 -> 62
- no-connect marks 1 -> 12
Other:
- note added: "Add Diode"
- note added: "Careful Vcc = 3.3V!!!!"
- note added: "Put USB-UART Transceiver on main carrier?\nMaybe on second carrier -> reduces cost -> USB not often used"
- moved on the sheet: U?
